File: KiCad/td-free.kicad_pcb (KiCad board)
At the start: 2 copper layers, 60 x 30 mm, 24 parts, among them J1 Conn_01x02_Pin, J2 USB_C_Receptacle_USB2.0_14P, Q1 2N7002, U1 ESP32-C3-WROOM-02, U2 VEML7700-TT, U3 AMS1117-3.3, U4 VEML3328, U5 TPD4E05U06DQA

Commit message: RGB LED Hardware
Parts:
- removed Q1: 2N7002, Package_TO_SOT_SMD:SOT-23
- added B1: Board, PCM_kikit:Board, F.Cu at (26.9, 25.1)
- added B2: Board, PCM_kikit:Board, F.Cu at (95.5, 24.9)
- added C7: 100nF, Capacitor_SMD:C_0805_2012Metric, B.Cu at (99.0, 29.4)
- added J3: 2mm 2x2 Receptacle, Connector_PinHeader_2.00mm:PinHeader_2x02_P2.00mm_Vertical_SMD, B.Cu at (106.0, 41.4)
- added LED1: XL-1615RGBC-WS2812B, easyeda2kicad:LED-SMD_4P-L1.6-W1.5_XL-1615RGBC-WS2812B-1, B.Cu at (98.8, 26.8)
- C1, C2, C3, C4, C5, C6: footprint Capacitor_SMD:C_0805_2012Metric_Pad1.18x1.45mm_HandSolder -> Capacitor_SMD:C_0805_2012Metric
- J1: value Conn_01x02_Pin -> 2mm 2x2 Header; footprint Connector_PinHeader_2.54mm:PinHeader_1x02_P2.54mm_Vertical -> easyeda2kicad:HDR-SMD_4P-P2.00-V-M-R2-C2-LS6.4-EH
- moved J1 25.1 mm to (62.5, 50.6), turned to 90 degrees
- moved C2 14.9 mm to (47.9, 29.1)
- moved C3 14.9 mm to (49.0, 36.1)
- moved C4 14.9 mm to (59.0, 38.1)
- moved C5 14.9 mm to (59.0, 34.1)
- moved C6 14.9 mm to (49.0, 41.1)
- moved D1 14.9 mm to (42.0, 40.1)
- moved R1 14.9 mm to (33.0, 32.1)
- moved TP1 14.9 mm to (59.0, 50.1)
- moved TP2 14.9 mm to (55.0, 50.0)
- moved TP3 14.9 mm to (51.0, 50.1)
- moved TP4 14.9 mm to (46.0, 50.1)
- moved TP5 14.9 mm to (41.0, 50.1)
- moved U3 14.9 mm to (40.1, 30.8)
- moved U1 14.9 mm to (69.9, 38.4)
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Connections:
- J1 pad 1: VBUS -> GND
- J1 pad 2: Net-(J1-Pin_2) -> GND
- U1 pad 6: /LED_C -> /MM_RGB
Routing:
- net VBUS: track 111.4 -> 68.2 mm
- net GND: track 24.3 -> 51.0 mm
- net Net-(J3-Pin_1): track 0.00 -> 24.0 mm
- net Net-(J1-Pin_2): track 21.4 -> 0.00 mm
- net /MM_RGB: track 0.00 -> 19.6 mm, vias 0 -> 2
- net Net-(J3-Pin_4): track 0.00 -> 18.8 mm
- net Net-(J3-Pin_3): track 0.00 -> 15.0 mm
- net /LED_C: track 12.4 -> 0.00 mm, vias 2 -> 0
- net Net-(U1-EN/CHIP_PU): track 18.3 -> 15.3 mm, vias 0 -> 2
- net /SDA1: track 7.86 -> 9.92 mm
- net /RGB_DATA: track 19.7 -> 21.4 mm
- net +3V3: track 61.0 -> 60.4 mm
Other:
- board size 60 x 30 mm -> 86.6 x 30.2 mm
- board text added: "Td-Free LED PCB V1"
- board text added: "V3.1"
- board text removed: "V2.1"
