File: KiCad/td-free.kicad_sch (KiCad schematic)
At the start: 24 parts, among them J1 Conn_01x02_Pin, J2 USB_C_Receptacle_USB2.0_14P, Q1 2N7002, U1 ESP32-C3-WROOM-02, U2 VEML7700-TT, U3 AMS1117-3.3, U4 VEML3328, U5 TPD4E05U06DQA

Commit message: RGB LED Hardware
Parts:
- removed J1: Conn_01x02_Pin, Connector_PinHeader_2.54mm:PinHeader_1x02_P2.54mm_Vertical, symbol Connector:Conn_01x02_Pin
- removed Q1: 2N7002, Package_TO_SOT_SMD:SOT-23, symbol Transistor_FET:2N7002
- added C7: 100nF, Capacitor_SMD:C_0805_2012Metric, symbol Device:C_Small
- added J1: 2mm 2x2 Header, easyeda2kicad:HDR-SMD_4P-P2.00-V-M-R2-C2-LS6.4-EH, symbol Connector_Generic:Conn_02x02_Counter_Clockwise
- added J3: 2mm 2x2 Receptacle, Connector_PinHeader_2.00mm:PinHeader_2x02_P2.00mm_Vertical_SMD, symbol Connector_Generic:Conn_02x02_Counter_Clockwise
- added LED1: XL-1615RGBC-WS2812B, easyeda2kicad:LED-SMD_4P-L1.6-W1.5_XL-1615RGBC-WS2812B-1, symbol easyeda2kicad:XL-1615RGBC-WS2812B
- C1, C2, C3, C4, C5, C6: footprint Capacitor_SMD:C_0805_2012Metric_Pad1.18x1.45mm_HandSolder -> Capacitor_SMD:C_0805_2012Metric
Connections:
- net GND: now also J1.1 (Pin_1), J1.2 (Pin_2)
- net VBUS: now also J1.4 (Pin_4)
- net LED_C renamed MM_RGB
- net MM_RGB: now also J1.3 (Pin_3)
- new net: C7.1, J3.1 (Pin_1), J3.2 (Pin_2), LED1.1 (GND)
- new net: J3.4 (Pin_4), LED1.2 (DIN)
- new net: C7.2, J3.3 (Pin_3), LED1.3 (VDD)
- no-connect marks 14 -> 15
Other:
- moved on the sheet: C3, C6, D1, D2, J2, R1, R2, U2, U4, U5
